File: hardware/sony-scopeman.kicad_pcb (KiCad board)
At the start: 2 copper layers, 53.5 x 101.8 mm, 135 parts, among them J1 EXT_X, J2 COIL_X, J3 EXT_Y, J4 COIL_Y, J5 SPEAKER, J6 USB_C_Receptacle_USB2.0, J7 BLK+CLK, J8 PWR, J9 GND, Q1 PZT3904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

Commit message: Make all Vectorboy files v1.3 to keep things aligned
Other:
- board text added: "v1.3"
- board text removed: "v1.0"
Changed lines of the file:
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@@
       (drillshape 0)
       (scaleselection 1)
-      (outputdirectory "gerber_V1.3"))
+      (outputdirectory "gerber-vectorboy-v1.3/"))
   )
   (net 0 "")
@@
     (add_net DAC_LRCK)
     (add_net ESP32_DAC0)
-    (add_net ESP32_DAC1)
     (add_net ESP32_FLASH)
     (add_net ESP32_PWM)
@@
     (add_net "Net-(R9-Pad2)")
     (add_net "Net-(SW1-Pad4)")
-    (add_net "Net-(U3-Pad17)")
-    (add_net "Net-(U3-Pad18)")
-    (add_net "Net-(U3-Pad19)")
-    (add_net "Net-(U3-Pad20)")
-    (add_net "Net-(U3-Pad21)")
-    (add_net "Net-(U3-Pad22)")
-    (add_net "Net-(U3-Pad23)")
-    (add_net "Net-(U3-Pad24)")
-    (add_net "Net-(U3-Pad26)")
-    (add_net "Net-(U3-Pad27)")
-    (add_net "Net-(U3-Pad28)")
-    (add_net "Net-(U3-Pad29)")
-    (add_net "Net-(U3-Pad32)")
-    (add_net "Net-(U3-Pad33)")
-    (add_net "Net-(U3-Pad4)")
-    (add_net "Net-(U3-Pad5)")
-    (add_net "Net-(U3-Pad8)")
-    (add_net "Net-(U3-Pad9)")
-    (add_net "Net-(U4-Pad2)")
     (add_net "Net-(U7-Pad1)")
     (add_net "Net-(U7-Pad10)")
@@
     (effects (font (size 1 0.7) (thickness 0.15)) (justify mirror))
   )
-  (gr_text v1.0 (at 142.748 102.616) (layer F.SilkS)
+  (gr_text v1.3 (at 142.748 102.616) (layer F.SilkS)
     (effects (font (size 1.2 1.2) (thickness 0.15)))
   )
